File: 2018/design/eagle/fri3d-badge-2018.brd (EAGLE design)
At the start: 80 x 75 mm, 64 parts

Commit message: unified values
Parts:
- C11, C9: value 100nF -> 0.1uF
- C6: value 47pf -> 47pF
- C8: value 10nF -> 0.01uF
- R1: value 64.9 -> 220
Changed lines of the file:
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@@
 <attribute name="VALUE" x="19.928" y="8.001" size="0.4064" layer="25" rot="R180"/>
 </element>
-<element name="C11" library="passive" package="0805" value="100nF" x="21.706" y="2.286" smashed="yes">
+<element name="C11" library="passive" package="0805" value="0.1uF" x="21.706" y="2.286" smashed="yes">
 <attribute name="NAME" x="19.293" y="2.3495" size="0.4064" layer="25"/>
 <attribute name="VALUE" x="18.785" y="1.651" size="0.4064" layer="25"/>
@@
 <attribute name="VALUE" x="37.973" y="2.656" size="0.4064" layer="25"/>
 </element>
-<element name="C6" library="passive" package="0805" value="47pf" x="11.303" y="17.261" smashed="yes">
+<element name="C6" library="passive" package="0805" value="47pF" x="11.303" y="17.261" smashed="yes">
 <attribute name="NAME" x="10.16" y="18.8485" size="0.4064" layer="25"/>
 <attribute name="VALUE" x="10.16" y="18.15" size="0.4064" layer="25"/>
@@
 <attribute name="VALUE" x="10.033" y="9.387" size="0.4064" layer="25"/>
 </element>
-<element name="C8" library="passive" package="0805" value="10nF" x="13.197" y="4.064" smashed="yes" rot="R90">
+<element name="C8" library="passive" package="0805" value="0.01uF" x="13.197" y="4.064" smashed="yes" rot="R90">
 <attribute name="NAME" x="13.6415" y="2.413" size="0.4064" layer="25" rot="R180"/>
 <attribute name="VALUE" x="14.594" y="3.048" size="0.4064" layer="25" rot="R90"/>
 </element>
-<element name="C9" library="passive" package="0805" value="100nF" x="14.097" y="9.387" smashed="yes" rot="R270">
+<element name="C9" library="passive" package="0805" value="0.1uF" x="14.097" y="9.387" smashed="yes" rot="R270">
 <attribute name="NAME" x="14.9225" y="10.149" size="0.4064" layer="25"/>
 <attribute name="VALUE" x="14.986" y="9.514" size="0.4064" layer="25"/>
@@
 <attribute name="SF_ID" value="PRT-08612" x="71.12" y="14.224" size="1.778" layer="28" rot="MR0" display="off"/>
 </element>
-<element name="R1" library="passive" package="0805" value="64.9" x="63.616" y="6.096" smashed="yes" rot="R90">
+<element name="R1" library="passive" package="0805" value="220" x="63.616" y="6.096" smashed="yes" rot="R90">
 <attribute name="NAME" x="65.2035" y="6.096" size="0.4064" layer="25" rot="R180"/>
 <attribute name="VALUE" x="65.648" y="5.461" size="0.4064" layer="25" rot="R180"/>
