File: 2018/design/eagle/fri3d-badge-2018.sch (EAGLE design)
At the start: 64 parts

Commit message: unified values
Parts:
- C11, C9: value 100nF -> 0.1uF
- C6: value 47pf -> 47pF
- C8: value 10nF -> 0.01uF
- R1: value 64.9 -> 220
Changed lines of the file:
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@@
 </classes>
 <parts>
-<part name="R1" library="passive" deviceset="RESISTOR" device="0805-RES" value="64.9"/>
+<part name="R1" library="passive" deviceset="RESISTOR" device="0805-RES" value="220"/>
 <part name="R2" library="passive" deviceset="RESISTOR" device="0805-RES" value="10K"/>
 <part name="C1" library="passive" deviceset="CAP" device="0805" value="4.7uF"/>
@@
 <part name="R3" library="passive" deviceset="RESISTOR" device="0805-RES" value="27"/>
 <part name="R4" library="passive" deviceset="RESISTOR" device="0805-RES" value="27"/>
-<part name="C6" library="passive" deviceset="CAP" device="0805" value="47pf"/>
+<part name="C6" library="passive" deviceset="CAP" device="0805" value="47pF"/>
 <part name="C7" library="passive" deviceset="CAP" device="0805" value="47pF"/>
 <part name="GND8" library="setup" deviceset="GND" device=""/>
-<part name="C8" library="passive" deviceset="CAP" device="0805" value="10nF"/>
+<part name="C8" library="passive" deviceset="CAP" device="0805" value="0.01uF"/>
 <part name="GND9" library="setup" deviceset="GND" device=""/>
-<part name="C9" library="passive" deviceset="CAP" device="0805" value="100nF"/>
+<part name="C9" library="passive" deviceset="CAP" device="0805" value="0.1uF"/>
 <part name="GND10" library="setup" deviceset="GND" device=""/>
 <part name="C10" library="passive" deviceset="CAP" device="0805" value="4.7uF"/>
-<part name="C11" library="passive" deviceset="CAP" device="0805" value="100nF"/>
+<part name="C11" library="passive" deviceset="CAP" device="0805" value="0.1uF"/>
 <part name="ESP32" library="esp32" deviceset="ESP-32S" device=""/>
 <part name="GND11" library="setup" deviceset="GND" device=""/>
